File: Hardware/PCB/28P-FPC-SPI-Debug.kicad_sch (KiCad schematic)
At the start: 40 parts, among them J1 Conn_01x08, J2 Conn_01x24, J3 SFV24R-1STBE1HLF, Q1 Si1308EDL, Q2 AO3401A, Q3 S8050, U1 RT9193-33GB, U2 TXB0108PW

Commit message: Modified FPC capacitor footprints to 0603 and 0805 due to production issues.
Parts:
- C1, C10, C13, C15, C16, C2, C3, C4, C5, C7, C9: footprint capacitors-cam:CAPC2012X140N -> Capacitor_SMD:C_0603_1608Metric_Pad1.08x0.95mm_HandSolder
- C11, C12: footprint capacitors-cam:CAPC2012X140N -> Capacitor_SMD:C_0805_2012Metric_Pad1.18x1.45mm_HandSolder
- J2: footprint Connector_PinHeader_2.54mm:PinHeader_2x12_P2.54mm_Vertical_SMD -> Connector_PinHeader_2.54mm:PinHeader_2x12_P2.54mm_Vertical
- Q3: footprint Package_TO_SOT_THT:TO-92_Inline -> mosfets:S8050
Changed lines of the file:
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@@
 			)
 		)
-		(property "Footprint" "Connector_PinHeader_2.54mm:PinHeader_2x12_P2.54mm_Vertical_SMD"
+		(property "Footprint" "Connector_PinHeader_2.54mm:PinHeader_2x12_P2.54mm_Vertical"
 			(at 274.32 132.08 0)
 			(effects
@@
 		(on_board yes)
 		(dnp no)
-		(fields_autoplaced yes)
 		(property "Reference" "C4"
 			(at 210.566 31.75 0)
@@
 			)
 		)
-		(property "Footprint" "capacitors-cam:CAPC2012X140N"
+		(property "Footprint" "Capacitor_SMD:C_0603_1608Metric_Pad1.08x0.95mm_HandSolder"
 			(at 208.28 30.48 0)
 			(effects
@@
 			)
 		)
-		(property "Footprint" "capacitors-cam:CAPC2012X140N"
+		(property "Footprint" "Capacitor_SMD:C_0603_1608Metric_Pad1.08x0.95mm_HandSolder"
 			(at 214.63 33.02 0)
 			(effects
@@
 			)
 		)
-		(property "Footprint" "Package_TO_SOT_THT:TO-92_Inline"
+		(property "Footprint" "mosfets:S8050"
 			(at 152.4 137.795 0)
 			(effects
@@
 			)
 		)
-		(property "Footprint" "capacitors-cam:CAPC2012X140N"
+		(property "Footprint" "Capacitor_SMD:C_0603_1608Metric_Pad1.08x0.95mm_HandSolder"
 			(at 241.3 64.77 0)
 			(effects
@@
 			)
 		)
-		(property "Footprint" "capacitors-cam:CAPC2012X140N"
+		(property "Footprint" "Capacitor_SMD:C_0805_2012Metric_Pad1.18x1.45mm_HandSolder"
 			(at 40.64 152.4 0)
 			(effects
@@
 			)
 		)
-		(property "Footprint" "capacitors-cam:CAPC2012X140N"
+		(property "Footprint" "Capacitor_SMD:C_0805_2012Metric_Pad1.18x1.45mm_HandSolder"
 			(at 60.96 165.1 0)
 			(effects
@@
 			)
 		)
-		(property "Footprint" "capacitors-cam:CAPC2012X140N"
+		(property "Footprint" "Capacitor_SMD:C_0603_1608Metric_Pad1.08x0.95mm_HandSolder"
 			(at 200.66 33.02 0)
 			(effects
@@
 			)
 		)
-		(property "Footprint" "capacitors-cam:CAPC2012X140N"
+		(property "Footprint" "Capacitor_SMD:C_0603_1608Metric_Pad1.08x0.95mm_HandSolder"
 			(at 241.3 91.44 0)
 			(effects
@@
 			)
 		)
-		(property "Footprint" "capacitors-cam:CAPC2012X140N"
+		(property "Footprint" "Capacitor_SMD:C_0603_1608Metric_Pad1.08x0.95mm_HandSolder"
 			(at 133.35 49.53 0)
 			(effects
@@
 			)
 		)
-		(property "Footprint" "capacitors-cam:CAPC2012X140N"
+		(property "Footprint" "Capacitor_SMD:C_0603_1608Metric_Pad1.08x0.95mm_HandSolder"
 			(at 237.49 33.02 0)
 			(effects
@@
 			)
 		)
-		(property "Footprint" "capacitors-cam:CAPC2012X140N"
+		(property "Footprint" "Capacitor_SMD:C_0603_1608Metric_Pad1.08x0.95mm_HandSolder"
 			(at 226.06 91.44 0)
 			(effects
@@
 			)
 		)
-		(property "Footprint" "capacitors-cam:CAPC2012X140N"
+		(property "Footprint" "Capacitor_SMD:C_0603_1608Metric_Pad1.08x0.95mm_HandSolder"
 			(at 92.71 34.29 0)
 			(effects
@@
 			)
 		)
-		(property "Footprint" "capacitors-cam:CAPC2012X140N"
+		(property "Footprint" "Capacitor_SMD:C_0603_1608Metric_Pad1.08x0.95mm_HandSolder"
 			(at 245.11 33.02 0)
 			(effects
@@
 			)
 		)
+		(property "Part No." ""
+			(at 245.11 31.75 0)
+			(effects
+				(font
+					(size 1.27 1.27)
+				)
+				(hide yes)
+			)
+		)
+		(property "Packaging" ""
+			(at 245.11 31.75 0)
+			(effects
+				(font
+					(size 1.27 1.27)
+				)
+				(hide yes)
+			)
+		)
 		(pin "2"
 		)
@@
 			)
 		)
-		(property "Footprint" "capacitors-cam:CAPC2012X140N"
+		(property "Footprint" "Capacitor_SMD:C_0603_1608Metric_Pad1.08x0.95mm_HandSolder"
 			(at 125.73 35.56 0)
 			(effects
